File: TJ_Quadrukopter/TJ_Quadrukopter.sch (KiCad schematic (older format))
At the start: 16 parts, among them M1 Motor_DC, M2 Motor_DC, M3 Motor_DC, M4 Motor_DC, Q1 IRF540N, Q2 IRF540N, Q3 IRF540N, Q4 IRF540N, U1 HC-06, U2 MPU6050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

Commit message: Added 3D models for arduino and connect them inside KiCADe, I have placed them before on differen drive path so maybe this will not shown correctly, but all used models and everything is here.
Parts:
- A1: footprint Module:Arduino_Nano -> LuboJ_footprints:Arduino_Nano; symbol MCU_Module:Arduino_Nano_v2.x -> LuboJ_parts:Arduino_Nano_v2.x
Changed lines of the file:
@@
 EESchema Schematic File Version 4
+LIBS:TJ_Quadrukopter-cache
 EELAYER 29 0
 EELAYER END
@@
 $EndDescr
 $Comp
-L MCU_Module:Arduino_Nano_v2.x A1
+L LuboJ_parts:Arduino_Nano_v2.x A1
 U 1 1 5EAAFDA2
 P 5850 4100
 F 0 "A1" V 5804 3057 50  0000 R CNN
 F 1 "Arduino_Nano_v2.x" V 5895 3057 50  0000 R CNN
-F 2 "Module:Arduino_Nano" H 6000 3150 50  0001 L CNN
+F 2 "LuboJ_footprints:Arduino_Nano" H 6000 3150 50  0001 L CNN
 F 3 "https://www.arduino.cc/en/uploads/Main/ArduinoNanoManual23.pdf" H 5850 3100 50  0001 C CNN
 	1    5850 4100
@@
 Wire Wire Line
 	5100 3200 5150 3200
-Connection ~ 6900 4400
 Wire Wire Line
 	4650 4200 4650 3200
 Wire Wire Line
-	6900 4300 6900 4400
-Wire Wire Line
 	4650 4200 4650 4800
 Wire Wire Line
+	4650 3200 5150 3200
+Wire Wire Line
 	6900 4300 6900 4900
-Wire Wire Line
-	4650 3200 5150 3200
 $EndSCHEMATC
